Commit message: Added joist mesh to repo and world file. Added dummy link to base in urdf

File: interbotix_ros_xshexapods/interbotix_xshexapod_descriptions/urdf/pxmark4.urdf.xacro (robot description, xacro)
@@ -130,4 +130,11 @@
     <link name="${robot_name}/${prefix}_foot_link"/>
   </xacro:macro>
+  <!-- Added to fix warning that root link can't have inertia in KDL -->
+  <link name="root"/>
+  <joint name="dummy_joint" type="fixed">
+    <origin rpy="0 0 0" xyz="0 0 0"/>
+    <parent link="root"/>
+    <child link="$(arg robot_name)/base_link"/>
+  </joint>
   <link name="$(arg robot_name)/base_link">
     <visual>

Commit message: Removing dummy link

File: interbotix_ros_xshexapods/interbotix_xshexapod_descriptions/urdf/pxmark4.urdf.xacro (robot description, xacro)
@@ -131,10 +131,10 @@
   </xacro:macro>
   <!-- Added to fix warning that root link can't have inertia in KDL -->
-  <link name="root"/>
+  <!-- <link name="root"/>
   <joint name="dummy_joint" type="fixed">
     <origin rpy="0 0 0" xyz="0 0 0"/>
     <parent link="root"/>
     <child link="$(arg robot_name)/base_link"/>
-  </joint>
+  </joint> -->
   <link name="$(arg robot_name)/base_link">
     <visual>

Commit message: Added 2 inch extension to urdf

File: interbotix_ros_xshexapods/interbotix_xshexapod_descriptions/urdf/pxmark4.urdf.xacro (robot description, xacro)
@@ -124,5 +124,5 @@
     </link>
     <joint name="${prefix}_foot" type="fixed">
-      <origin rpy="0 0 0" xyz="0.095 0 -0.09"/>
+      <origin rpy="0 0 0" xyz="0.13067 0 -0.1238"/>
       <parent link="${robot_name}/${prefix}_tibia_link"/>
       <child link="${robot_name}/${prefix}_foot_link"/>

Commit message: Reverting unnecessary changes

File: interbotix_ros_xshexapods/interbotix_xshexapod_descriptions/urdf/pxmark4.urdf.xacro (robot description, xacro)
@@ -130,11 +130,4 @@
     <link name="${robot_name}/${prefix}_foot_link"/>
   </xacro:macro>
-  <!-- Added to fix warning that root link can't have inertia in KDL -->
-  <!-- <link name="root"/>
-  <joint name="dummy_joint" type="fixed">
-    <origin rpy="0 0 0" xyz="0 0 0"/>
-    <parent link="root"/>
-    <child link="$(arg robot_name)/base_link"/>
-  </joint> -->
   <link name="$(arg robot_name)/base_link">
     <visual>
