Commit message: edit urdf to add new joints

File: interbotix_ros_xshexapods/interbotix_xshexapod_descriptions/urdf/wxmark4.urdf.xacro (robot description, xacro)
@@ -11,4 +11,128 @@
     <texture filename="package://interbotix_xshexapod_descriptions/meshes/interbotix_black.png"/>
   </material>
+  <joint name="turret_rot" type="revolute">
+    <axis xyz="0 0 1"/>
+    <limit effort="3" lower="${radians(-90)}" upper="${radians(90)}" velocity="${pi}"/>
+    <origin rpy="0 0 0" xyz="0 0 .23"/>
+    <parent link="${robot_name}/base_link"/>
+    <child link="${robot_name}/turret_rot_link"/>
+  </joint>
+  <transmission name="trans_turret_rot">
+    <type>transmission_interface/SimpleTransmission</type>
+    <joint name="$turret_rot">
+      <hardwareInterface>hardware_interface/EffortJointInterface</hardwareInterface>
+    </joint>
+    <actuator name="$turret_rot_motor">
+      <mechanicalReduction>1</mechanicalReduction>
+    </actuator>
+  </transmission>
+  <link name="${robot_name}/turret_rot_link">
+    <visual>
+      <origin rpy="0 0 0" xyz="0 0 0"/>
+      <geometry>
+        <cylinder radius=".05" length="0.23"/>
+      </geometry>
+      <material name="interbotix_black"/>
+    </visual>
+    <collision>
+      <origin rpy="0 0 0" xyz="0 0 0"/>
+      <geometry>
+        <cylinder radius=".05" length="0.23"/>
+      </geometry>
+    </collision>
+  </link>
+  <joint name="turret_ext" type="prismatic">
+    <axis xyz="1 0 0"/>
+    <limit effort="3" lower="0" upper=".25" velocity="1"/>
+    <origin rpy="0 0 0" xyz="0 0 0"/>
+    <parent link="${robot_name}/turret_rot_link"/>
+    <child link="${robot_name}/turret_ext_link"/>
+  </joint>
+  <transmission name="trans_turret_ext">
+    <type>transmission_interface/SimpleTransmission</type>
+    <joint name="$turret_ext">
+      <hardwareInterface>hardware_interface/EffortJointInterface</hardwareInterface>
+    </joint>
+    <actuator name="$turret_ext_motor">
+      <mechanicalReduction>1</mechanicalReduction>
+    </actuator>
+  </transmission>
+  <link name="${robot_name}/turret_ext_link">
+    <visual>
+      <origin rpy="0 0 0" xyz="0 0 0"/>
+      <geometry>
+        <cylinder radius=".05" length="0.15"/>
+      </geometry>
+      <material name="interbotix_black"/>
+    </visual>
+    <collision>
+      <origin rpy="0 0 0" xyz="0 0 0"/>
+      <geometry>
+        <cylinder radius=".05" length="0.15"/>
+      </geometry>
+    </collision>
+  </link>
+  <joint name="turret_tilt" type="revolute">
+    <axis xyz="0 1 0"/>
+    <limit effort="3" lower="${radians(-60)}" upper="${radians(60)}" velocity="1"/>
+    <origin rpy="0 0 0" xyz="0 0 0"/>
+    <parent link="${robot_name}/turret_ext_link"/>
+    <child link="${robot_name}/turret_tilt_link"/>
+  </joint>
+  <transmission name="trans_turret_tilt">
+    <type>transmission_interface/SimpleTransmission</type>
+    <joint name="$turret_tilt">
+      <hardwareInterface>hardware_interface/EffortJointInterface</hardwareInterface>
+    </joint>
+    <actuator name="$turret_tilt_motor">
+      <mechanicalReduction>1</mechanicalReduction>
+    </actuator>
+  </transmission>
+  <link name="${robot_name}/turret_tilt_link">
+    <visual>
+      <origin rpy="0 0 0" xyz="0 0 0"/>
+      <geometry>
+        <cylinder radius=".05" length="0.23"/>
+      </geometry>
+      <material name="interbotix_black"/>
+    </visual>
+    <collision>
+      <origin rpy="0 0 0" xyz="0 0 0"/>
+      <geometry>
+        <cylinder radius=".05" length="0.23"/>
+      </geometry>
+    </collision>
+  </link>
+  <joint name="turret_pinch" type="prismatic">
+    <axis xyz="0 1 0"/>
+    <limit effort="3" lower="0" upper=".005" velocity="1"/>
+    <origin rpy="0 0 0" xyz="0 0 0"/>
+    <parent link="${robot_name}/turret_tilt_link"/>
+    <child link="${robot_name}/turret_pinch_link"/>
+  </joint>
+  <transmission name="trans_turret_pinch">
+    <type>transmission_interface/SimpleTransmission</type>
+    <joint name="$turret_tilt">
+      <hardwareInterface>hardware_interface/EffortJointInterface</hardwareInterface>
+    </joint>
+    <actuator name="$turret_pinch_motor">
+      <mechanicalReduction>1</mechanicalReduction>
+    </actuator>
+  </transmission>
+  <link name="${robot_name}/turret_pinch_link">
+    <visual>
+      <origin rpy="0 0 0" xyz="0 0 0"/>
+      <geometry>
+        <cylinder radius=".01" length="0.01"/>
+      </geometry>
+      <material name="interbotix_black"/>
+    </visual>
+    <collision>
+      <origin rpy="0 0 0" xyz="0 0 0"/>
+      <geometry>
+        <cylinder radius=".01" length="0.01"/>
+      </geometry>
+    </collision>
+  </link>
   <xacro:macro name="leg" params="robot_name prefix x y yaw">
     <joint name="${prefix}_coxa" type="revolute">

Commit message: fix urdf new motor gen

File: interbotix_ros_xshexapods/interbotix_xshexapod_descriptions/urdf/wxmark4.urdf.xacro (robot description, xacro)
@@ -20,8 +20,8 @@
   <transmission name="trans_turret_rot">
     <type>transmission_interface/SimpleTransmission</type>
-    <joint name="$turret_rot">
-      <hardwareInterface>hardware_interface/EffortJointInterface</hardwareInterface>
-    </joint>
-    <actuator name="$turret_rot_motor">
+    <joint name="turret_rot">
+      <hardwareInterface>hardware_interface/EffortJointInterface</hardwareInterface>
+    </joint>
+    <actuator name="turret_rot_motor">
       <mechanicalReduction>1</mechanicalReduction>
     </actuator>
@@ -51,8 +51,8 @@
   <transmission name="trans_turret_ext">
     <type>transmission_interface/SimpleTransmission</type>
-    <joint name="$turret_ext">
-      <hardwareInterface>hardware_interface/EffortJointInterface</hardwareInterface>
-    </joint>
-    <actuator name="$turret_ext_motor">
+    <joint name="turret_ext">
+      <hardwareInterface>hardware_interface/EffortJointInterface</hardwareInterface>
+    </joint>
+    <actuator name="turret_ext_motor">
       <mechanicalReduction>1</mechanicalReduction>
     </actuator>
@@ -82,8 +82,8 @@
   <transmission name="trans_turret_tilt">
     <type>transmission_interface/SimpleTransmission</type>
-    <joint name="$turret_tilt">
-      <hardwareInterface>hardware_interface/EffortJointInterface</hardwareInterface>
-    </joint>
-    <actuator name="$turret_tilt_motor">
+    <joint name="turret_tilt">
+      <hardwareInterface>hardware_interface/EffortJointInterface</hardwareInterface>
+    </joint>
+    <actuator name="turret_tilt_motor">
       <mechanicalReduction>1</mechanicalReduction>
     </actuator>
@@ -113,8 +113,8 @@
   <transmission name="trans_turret_pinch">
     <type>transmission_interface/SimpleTransmission</type>
-    <joint name="$turret_tilt">
-      <hardwareInterface>hardware_interface/EffortJointInterface</hardwareInterface>
-    </joint>
-    <actuator name="$turret_pinch_motor">
+    <joint name="turret_tilt">
+      <hardwareInterface>hardware_interface/EffortJointInterface</hardwareInterface>
+    </joint>
+    <actuator name="turret_pinch_motor">
       <mechanicalReduction>1</mechanicalReduction>
     </actuator>

Commit message: control turret from ps4

File: interbotix_ros_xshexapods/interbotix_xshexapod_descriptions/urdf/wxmark4.urdf.xacro (robot description, xacro)
@@ -15,6 +15,6 @@
     <limit effort="3" lower="${radians(-90)}" upper="${radians(90)}" velocity="${pi}"/>
     <origin rpy="0 0 0" xyz="0 0 .23"/>
-    <parent link="${robot_name}/base_link"/>
-    <child link="${robot_name}/turret_rot_link"/>
+    <parent link="$(arg robot_name)/base_link"/>
+    <child link="$(arg robot_name)/turret_rot_link"/>
   </joint>
   <transmission name="trans_turret_rot">
@@ -27,5 +27,5 @@
     </actuator>
   </transmission>
-  <link name="${robot_name}/turret_rot_link">
+  <link name="$(arg robot_name)/turret_rot_link">
     <visual>
       <origin rpy="0 0 0" xyz="0 0 0"/>
@@ -46,6 +46,6 @@
     <limit effort="3" lower="0" upper=".25" velocity="1"/>
     <origin rpy="0 0 0" xyz="0 0 0"/>
-    <parent link="${robot_name}/turret_rot_link"/>
-    <child link="${robot_name}/turret_ext_link"/>
+    <parent link="$(arg robot_name)/turret_rot_link"/>
+    <child link="$(arg robot_name)/turret_ext_link"/>
   </joint>
   <transmission name="trans_turret_ext">
@@ -58,5 +58,5 @@
     </actuator>
   </transmission>
-  <link name="${robot_name}/turret_ext_link">
+  <link name="$(arg robot_name)/turret_ext_link">
     <visual>
       <origin rpy="0 0 0" xyz="0 0 0"/>
@@ -77,6 +77,6 @@
     <limit effort="3" lower="${radians(-60)}" upper="${radians(60)}" velocity="1"/>
     <origin rpy="0 0 0" xyz="0 0 0"/>
-    <parent link="${robot_name}/turret_ext_link"/>
-    <child link="${robot_name}/turret_tilt_link"/>
+    <parent link="$(arg robot_name)/turret_ext_link"/>
+    <child link="$(arg robot_name)/turret_tilt_link"/>
   </joint>
   <transmission name="trans_turret_tilt">
@@ -89,5 +89,5 @@
     </actuator>
   </transmission>
-  <link name="${robot_name}/turret_tilt_link">
+  <link name="$(arg robot_name)/turret_tilt_link">
     <visual>
       <origin rpy="0 0 0" xyz="0 0 0"/>
@@ -108,6 +108,6 @@
     <limit effort="3" lower="0" upper=".005" velocity="1"/>
     <origin rpy="0 0 0" xyz="0 0 0"/>
-    <parent link="${robot_name}/turret_tilt_link"/>
-    <child link="${robot_name}/turret_pinch_link"/>
+    <parent link="$(arg robot_name)/turret_tilt_link"/>
+    <child link="$(arg robot_name)/turret_pinch_link"/>
   </joint>
   <transmission name="trans_turret_pinch">
@@ -120,5 +120,5 @@
     </actuator>
   </transmission>
-  <link name="${robot_name}/turret_pinch_link">
+  <link name="$(arg robot_name)/turret_pinch_link">
     <visual>
       <origin rpy="0 0 0" xyz="0 0 0"/>

Commit message: Added 2 inch leg extension to urdf

File: interbotix_ros_xshexapods/interbotix_xshexapod_descriptions/urdf/wxmark4.urdf.xacro (robot description, xacro)
@@ -245,5 +245,6 @@
     </link>
     <joint name="${prefix}_foot" type="fixed">
-      <origin rpy="0 0 0" xyz="0.095 0 -0.09"/>
+      <!-- <origin rpy="0 0 0" xyz="0.095 0 -0.09"/> -->
+      <origin rpy="0 0 0" xyz="0.13067 0 -0.1238"/>
       <parent link="${robot_name}/${prefix}_tibia_link"/>
       <child link="${robot_name}/${prefix}_foot_link"/>

Commit message: previous changes

File: interbotix_ros_xshexapods/interbotix_xshexapod_descriptions/urdf/wxmark4.urdf.xacro (robot description, xacro)
@@ -247,4 +247,5 @@
       <!-- <origin rpy="0 0 0" xyz="0.095 0 -0.09"/> -->
       <origin rpy="0 0 0" xyz="0.13067 0 -0.1238"/>
+      <!-- <origin rpy="0 0 0" xyz="0.16634 0 -0.1576"/> -->
       <parent link="${robot_name}/${prefix}_tibia_link"/>
       <child link="${robot_name}/${prefix}_foot_link"/>
